File: hardware/OpenAVNS KiCad Project.kicad_pcb (KiCad board)
At the start: 2 copper layers, 164 parts, among them J1 Conn_ARM_JTAG_SWD_10, J2 USB_C_Receptacle, J3 Conn_01x02_Pin, Q1 BCV62, Q2 BC847, Q3 BC857, Q4 BCV61, Q5 BCV62, Q6 BC847, Q7 BC857, Q8 BCV61, SW1 SW_SPDT, T2 Wurth 750315839 - 1:10, 40uH, U1 TS5A3159AYZPR, U10 OPA455, U11 LIS2DH12, U12 OPA455, U13 74AUC1G74, U14 TPS61200DRC, U16 LT1615ES5_TRPBF, U17 LT8304IS8E_PBF, U18 MCP73831-2-OT, U2 TLV9004xRUCR, U3 MCP4725xxx-xCH, U4 TS5A3159AYZPR, U5 nRF52840, U6 TS5A3159AYZPR, U7 MCP4725xxx-xCH, U8 TS5A3159AYZPR, U9 TLV9062, Y1 32MHz

Commit message: Fixed some schematic parts, added test points and 3.5mm jack for output
Parts:
- removed C50: 22uF, 200V, Capacitor_SMD:C_1210_3225Metric
- removed C52, C53: C_Polarized_US, Capacitor_THT:CP_Radial_D12.5mm_P5.00mm
- removed R67: 1k, Resistor_SMD:R_0402_1005Metric
- removed R68: 2k, Resistor_SMD:R_0402_1005Metric
- removed T2: Wurth 750315839 - 1:10, 40uH, OpenAVNS:WE-FLYLT_EP13_5465
- removed U18: MCP73831-2-OT, Package_TO_SOT_SMD:SOT-23-5
- added AT1: 2450AT43B100E, OpenAVNS:ANTENNA_2450AT43B100E, F.Cu at (58.5, 99.8)
- added C29: 10uF, Capacitor_SMD:C_0603_1608Metric, F.Cu at (82.9, 78.3)
- added C30: 100nF, Capacitor_SMD:C_0402_1005Metric, F.Cu at (60.9, 73.0)
- added C49: 4.7uF, Capacitor_SMD:C_0805_2012Metric, F.Cu at (74.4, 36.4)
- added J4: Conn_01x02_Pin, Connector_PinHeader_2.00mm:PinHeader_1x02_P2.00mm_Vertical, F.Cu at (90.9, 74.0)
- added R52: 0 Ohm, Resistor_SMD:R_0603_1608Metric_Pad0.98x0.95mm_HandSolder, F.Cu at (46.7, 85.8)
- added R55: 0 Ohm, Resistor_SMD:R_0603_1608Metric_Pad0.98x0.95mm_HandSolder, F.Cu at (46.7, 93.3)
- added T1: Wurth 750315839 - 1:10, 40uH, OpenAVNS:WE-FLYLT_EP13_5465, F.Cu at (60.2, 41.8)
- added TP1: TestPoint, TestPoint:TestPoint_Pad_D2.0mm, F.Cu at (26.3, 34.0)
- added TP10: TestPoint, TestPoint:TestPoint_Pad_D2.0mm, F.Cu at (30.3, 38.0)
- added TP11: TestPoint, TestPoint:TestPoint_Pad_D2.0mm, F.Cu at (30.3, 42.1)
- added TP12: TestPoint, TestPoint:TestPoint_Pad_D2.0mm, F.Cu at (30.3, 46.1)
- added TP13: TestPoint, TestPoint:TestPoint_Pad_D2.0mm, F.Cu at (30.3, 50.2)
- added TP14: TestPoint, TestPoint:TestPoint_Pad_D2.0mm, F.Cu at (30.3, 54.2)
- added TP15: TestPoint, TestPoint:TestPoint_Pad_D2.0mm, F.Cu at (30.3, 58.3)
- added TP16: TestPoint, TestPoint:TestPoint_Pad_D2.0mm, F.Cu at (30.3, 62.3)
- added TP17: TestPoint, TestPoint:TestPoint_Pad_D2.0mm, F.Cu at (34.4, 34.0)
- added TP18: TestPoint, TestPoint:TestPoint_Pad_D2.0mm, F.Cu at (34.4, 38.0)
- added TP19: TestPoint, TestPoint:TestPoint_Pad_D2.0mm, F.Cu at (34.4, 42.1)
- added TP2: TestPoint, TestPoint:TestPoint_Pad_D2.0mm, F.Cu at (26.3, 38.0)
- added TP20: TestPoint, TestPoint:TestPoint_Pad_D2.0mm, F.Cu at (34.4, 46.1)
- added TP21: TestPoint, TestPoint:TestPoint_Pad_D2.0mm, F.Cu at (34.4, 50.2)
- added TP22: TestPoint, TestPoint:TestPoint_Pad_D2.0mm, F.Cu at (34.4, 54.2)
- added TP23: TestPoint, TestPoint:TestPoint_Pad_D2.0mm, F.Cu at (34.4, 58.3)
- added TP24: TestPoint, TestPoint:TestPoint_Pad_D2.0mm, F.Cu at (34.4, 62.3)
- added TP25: TestPoint, TestPoint:TestPoint_Pad_D2.0mm, F.Cu at (38.4, 34.0)
- added TP26: TestPoint, TestPoint:TestPoint_Pad_D2.0mm, F.Cu at (38.4, 38.0)
- added TP27: TestPoint, TestPoint:TestPoint_Pad_D2.0mm, F.Cu at (38.4, 42.1)
- added TP28: TestPoint, TestPoint:TestPoint_Pad_D2.0mm, F.Cu at (38.4, 46.1)
- added TP29: TestPoint, TestPoint:TestPoint_Pad_D2.0mm, F.Cu at (38.4, 50.2)
- added TP3: TestPoint, TestPoint:TestPoint_Pad_D2.0mm, F.Cu at (26.3, 42.1)
- added TP30: TestPoint, TestPoint:TestPoint_Pad_D2.0mm, F.Cu at (38.4, 54.2)
- added TP31: TestPoint, TestPoint:TestPoint_Pad_D2.0mm, F.Cu at (38.4, 58.3)
- added TP32: TestPoint, TestPoint:TestPoint_Pad_D2.0mm, F.Cu at (38.4, 62.3)
- added TP33: TestPoint, TestPoint:TestPoint_Pad_D2.0mm, F.Cu at (42.5, 34.0)
- added TP34: TestPoint, TestPoint:TestPoint_Pad_D2.0mm, F.Cu at (42.5, 38.0)
- added TP35: TestPoint, TestPoint:TestPoint_Pad_D2.0mm, F.Cu at (42.5, 42.1)
- added TP36: TestPoint, TestPoint:TestPoint_Pad_D2.0mm, F.Cu at (42.5, 46.1)
- added TP37: TestPoint, TestPoint:TestPoint_Pad_D2.0mm, F.Cu at (42.5, 50.2)
- added TP38: TestPoint, TestPoint:TestPoint_Pad_D2.0mm, F.Cu at (42.5, 54.2)
- added TP39: TestPoint, TestPoint:TestPoint_Pad_D2.0mm, F.Cu at (42.5, 58.3)
- added TP4: TestPoint, TestPoint:TestPoint_Pad_D2.0mm, F.Cu at (26.3, 46.1)
- added TP40: TestPoint, TestPoint:TestPoint_Pad_D2.0mm, F.Cu at (42.5, 62.3)
- added TP5: TestPoint, TestPoint:TestPoint_Pad_D2.0mm, F.Cu at (26.3, 50.2)
- added TP6: TestPoint, TestPoint:TestPoint_Pad_D2.0mm, F.Cu at (26.3, 54.2)
- added TP7: TestPoint, TestPoint:TestPoint_Pad_D2.0mm, F.Cu at (26.3, 58.3)
- added TP8: TestPoint, TestPoint:TestPoint_Pad_D2.0mm, F.Cu at (26.3, 62.3)
- added TP9: TestPoint, TestPoint:TestPoint_Pad_D2.0mm, F.Cu at (30.3, 34.0)
- added U15: LT1615ES5_TRPBF, OpenAVNS:SOT95P280X145-5N, F.Cu at (79.5, 101.3)
- C15: value 22uF -> 22uF, 100V
- C16: value 680pF -> 22uF, 100V; footprint Capacitor_SMD:C_0402_1005Metric -> Capacitor_SMD:C_1210_3225Metric
- C17: value 12pF -> 22uF; footprint Capacitor_SMD:C_0402_1005Metric -> Capacitor_SMD:C_1210_3225Metric
- C18: value 100nF -> 10uF; footprint Capacitor_SMD:C_0402_1005Metric -> Capacitor_SMD:C_0603_1608Metric
- C19: value 22uF -> 100nF; footprint Capacitor_SMD:C_1210_3225Metric -> Capacitor_SMD:C_0402_1005Metric
- C20: value 100nF -> 680pF
- C21: value 100nF -> 12pF
- C22: value 10uF -> 100nF; footprint Capacitor_SMD:C_0603_1608Metric -> Capacitor_SMD:C_0402_1005Metric
- C23: value 0.1uF -> 22uF; footprint Capacitor_SMD:C_0603_1608Metric -> Capacitor_SMD:C_1210_3225Metric
- C24: value 10uF -> 100nF; footprint Capacitor_SMD:C_0805_2012Metric -> Capacitor_SMD:C_0402_1005Metric
- C25: value 0.1uF -> 100nF; footprint Capacitor_SMD:C_0603_1608Metric -> Capacitor_SMD:C_0402_1005Metric
- C26: value 22uF -> 10uF; footprint Capacitor_SMD:C_0805_2012Metric -> Capacitor_SMD:C_0603_1608Metric
- C27: value 22uF, 100V -> 100nF; footprint Capacitor_SMD:C_1210_3225Metric -> Capacitor_SMD:C_0402_1005Metric
- C28: value 1uF -> 10uF; footprint Capacitor_SMD:C_0805_2012Metric -> Capacitor_SMD:C_0603_1608Metric
- C31: value 22uF, 200V -> 0.1uF; footprint Capacitor_SMD:C_1210_3225Metric -> Capacitor_SMD:C_0603_1608Metric
- C32: value 1uF -> 10uF
- C33: value 22uF, 50V -> 0.1uF; footprint Capacitor_SMD:C_0805_2012Metric -> Capacitor_SMD:C_0603_1608Metric
- C34: value 4.7pF -> 22uF
- C35: value 22uF -> 22uF, 100V; footprint Capacitor_SMD:C_0805_2012Metric -> Capacitor_SMD:C_1210_3225Metric
- C36: value 22uF, 100V -> 1uF; footprint Capacitor_SMD:C_1210_3225Metric -> Capacitor_SMD:C_0805_2012Metric
- C37: value 10pF -> 22uF, 200V; footprint Capacitor_SMD:C_0603_1608Metric -> Capacitor_SMD:C_1210_3225Metric
- C38: value 1uF -> C_Polarized_US; footprint Capacitor_SMD:C_0603_1608Metric -> Capacitor_THT:CP_Radial_D12.5mm_P5.00mm
- C39: value 4.7uF -> 1uF
- C40: value 4.7uF -> 22uF, 200V; footprint Capacitor_SMD:C_0805_2012Metric -> Capacitor_SMD:C_1210_3225Metric
- C41: value 100nF -> C_Polarized_US; footprint Capacitor_SMD:C_0402_1005Metric -> Capacitor_THT:CP_Radial_D12.5mm_P5.00mm
- C42: value 100nF -> 22uF, 50V; footprint Capacitor_SMD:C_0402_1005Metric -> Capacitor_SMD:C_0805_2012Metric
- C43: value 10uF -> 4.7pF; footprint Capacitor_SMD:C_0603_1608Metric -> Capacitor_SMD:C_0805_2012Metric
- C44: value 10uF -> 22uF; footprint Capacitor_SMD:C_0603_1608Metric -> Capacitor_SMD:C_0805_2012Metric
- C46: value 22uF, 100V -> 1uF; footprint Capacitor_SMD:C_1210_3225Metric -> Capacitor_SMD:C_0603_1608Metric
- C47: value 100nF -> 10pF; footprint Capacitor_SMD:C_0402_1005Metric -> Capacitor_SMD:C_0603_1608Metric
- C48: value 10uF -> 4.7uF; footprint Capacitor_SMD:C_0603_1608Metric -> Capacitor_SMD:C_0805_2012Metric
- D11: value MBR0530 -> SS3200; footprint Diode_SMD:D_SOD-123 -> Diode_SMD:D_SMA
- D12: value LED Yellow -> MBR0530; footprint LED_SMD:LED_0402_1005Metric -> Diode_SMD:D_SOD-123
- D13: value LED Green -> LED Yellow
- D14: value SS3200 -> LED Green; footprint Diode_SMD:D_SMA -> LED_SMD:LED_0402_1005Metric
- J2: value USB_C_Receptacle -> AudioPlug3; footprint Connector_USB:USB_C_Receptacle_Amphenol_12401548E4-2A -> Connector_Audio:Jack_3.5mm_CUI_SJ-3523-SMT_Horizontal
- J3: value Conn_01x02_Pin -> USB_C_Receptacle; footprint Connector_PinHeader_2.00mm:PinHeader_1x02_P2.00mm_Vertical -> Connector_USB:USB_C_Receptacle_Amphenol_12401548E4-2A
- R56: value 0 Ohm -> 100k; footprint Resistor_SMD:R_0603_1608Metric_Pad0.98x0.95mm_HandSolder -> Resistor_SMD:R_0805_2012Metric_Pad1.20x1.40mm_HandSolder
- R57: value 0 Ohm -> 2M; footprint Resistor_SMD:R_0603_1608Metric_Pad0.98x0.95mm_HandSolder -> Resistor_SMD:R_0603_1608Metric
- R58: footprint Resistor_SMD:R_0805_2012Metric_Pad1.20x1.40mm_HandSolder -> Resistor_SMD:R_0402_1005Metric
- R59: value 2M -> 100k; footprint Resistor_SMD:R_0603_1608Metric -> Resistor_SMD:R_0402_1005Metric
- R60: value 100k -> 0 Ohm; footprint Resistor_SMD:R_0402_1005Metric -> Resistor_SMD:R_0603_1608Metric_Pad0.98x0.95mm_HandSolder
- R61: value 100k -> 10k; footprint Resistor_SMD:R_0402_1005Metric -> Resistor_SMD:R_0805_2012Metric_Pad1.20x1.40mm_HandSolder
- R62: value 0 Ohm -> 130k; footprint Resistor_SMD:R_0603_1608Metric_Pad0.98x0.95mm_HandSolder -> Resistor_SMD:R_0603_1608Metric
- R63: value 10k -> 330; footprint Resistor_SMD:R_0805_2012Metric_Pad1.20x1.40mm_HandSolder -> Resistor_SMD:R_0402_1005Metric
- R64: value 130k -> 100k; footprint Resistor_SMD:R_0603_1608Metric -> Resistor_SMD:R_0402_1005Metric
- R65: value 330 -> 1k
- R66: value 100k -> 2k
- U10: value OPA455 -> TLV9062; footprint Package_SO:TI_SO-PowerPAD-8_ThermalVias -> OpenAVNS:QFN50P200X150X40-10N
- U16: value LT1615ES5_TRPBF -> LT8304IS8E_PBF; footprint OpenAVNS:SOT95P280X145-5N -> OpenAVNS:SOIC127P599X175-9N
- U17: value LT8304IS8E_PBF -> MCP73831-2-OT; footprint OpenAVNS:SOIC127P599X175-9N -> Package_TO_SOT_SMD:SOT-23-5
- U9: value TLV9062 -> OPA455; footprint OpenAVNS:QFN50P200X150X40-10N -> Package_SO:TI_SO-PowerPAD-8_ThermalVias
- Y1: value 32MHz -> 32MHz - X322532MOB4SI; footprint Crystal:Crystal_SMD_2016-4Pin_2.0x1.6mm -> Crystal:Crystal_SMD_3225-4Pin_3.2x2.5mm
- moved D14 85.8 mm to (91.1, 57.8)
- moved S1 84.8 mm to (85.3, 54.2)
- moved L3 77.6 mm to (29.0, 96.9)
- moved U17 77.1 mm to (41.2, 76.0)
- moved U16 70.6 mm to (57.4, 54.9)
- moved SW1 67.8 mm to (84.0, 64.3)
- moved D11 64.5 mm to (48.6, 57.0)
- moved C48 63.8 mm to (74.4, 33.4)
- moved C38 63.2 mm to (29.1, 71.4)
- moved J2 57.6 mm to (87.2, 41.5)
- moved C43 56.7 mm to (70.0, 48.5)
- moved C41 54.4 mm to (29.1, 85.4)
- moved U4 54.1 mm to (67.4, 66.1)
- moved U1 54.1 mm to (63.5, 66.1)
- moved U6 54.1 mm to (71.4, 66.1)
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Connections:
- C15 pad 1: /E2_Pre -> /+HV
- C15 pad 2: /E2 -> GND
- C16 pad 1: /E2_Pre -> /-HV
- C17 pad 1: Net-(U5-XC2) -> /E2_Pre
- C17 pad 2: GND -> /E2
- C19 pad 1: GND -> +3.3V
- C19 pad 2: /Ground_Electrode -> GND
- C20 pad 1: +3.3V -> /E2_Pre
- C21 pad 1: +3.3V -> Net-(U5-XC2)
- C23 pad 1: /V_ON -> GND
- C23 pad 2: Net-(U14-UVLO) -> /Ground_Electrode
- C24 pad 1: /V_ON -> +3.3V
- C25 pad 1: Net-(U14-VAUX) -> +3.3V
- C27 pad 1: /-20V -> +3.3V
- C28 pad 1: Net-(D7-K) -> +3.3V
- C28 pad 2: Net-(U16-SW) -> GND
- C31 pad 1: /+50V -> /V_ON
- C31 pad 2: GND -> Net-(U14-UVLO)
- C32 pad 1: Net-(U16-SW) -> /V_ON
- C32 pad 2: Net-(D10-A) -> GND
- C33 pad 1: /V_ON -> Net-(U14-VAUX)
- C34 pad 1: /+20V -> +3.3V
- C34 pad 2: /20V_FB -> GND
- C35 pad 1: /V_ON -> /-20V
- C36 pad 1: /+20V -> Net-(D7-K)
- C36 pad 2: GND -> Net-(U15-SW)
- C37 pad 1: Net-(U17-RREF) -> /+50V
- C38 pad 1: Net-(U17-INTVCC) -> /+50V
- C39 pad 1: /V_USB -> Net-(U15-SW)
- C39 pad 2: GND -> Net-(D10-A)
- C40 pad 1: /VBAT -> GND
- C40 pad 2: GND -> /-50V
- C41 pad 1: +3.3V -> GND
- C41 pad 2: GND -> /-50V
- C42 pad 1: +3.3V -> /V_ON
- C43 pad 1: +3.3V -> /+20V
- C43 pad 2: GND -> /20V_FB
- C44 pad 1: +3.3V -> /V_ON
- C45 pad 1: /+HV -> /+20V
- C46 pad 1: /-HV -> Net-(U16-INTVCC)
- C47 pad 1: +3.3V -> Net-(U16-RREF)
- C48 pad 1: +3.3V -> /V_USB
- D11 pad 1: Net-(D10-A) -> Net-(D11-K)
- D11 pad 2: GND -> /-50V
- D12 pad 1: Net-(D12-K) -> Net-(D10-A)
- D12 pad 2: /V_USB -> GND
- D13 pad 2: /V_ON -> /V_USB
- D14 pad 2: /-50V -> /V_ON
- L3 pad 2: Net-(U16-SW) -> Net-(U15-SW)
- R34 pad 2: Net-(U9A--) -> Net-(U10A--)
- R35 pad 1: Net-(U9A--) -> Net-(U10A--)
- R36 pad 2: Net-(J2-CC1) -> Net-(J3-CC1)
- R37 pad 2: Net-(J2-CC2) -> Net-(J3-CC2)
- R39 pad 1: Net-(U9A--) -> Net-(U10A--)
- R41 pad 2: Net-(U9B--) -> Net-(U10B--)
- R42 pad 1: Net-(U9B--) -> Net-(U10B--)
- R45 pad 1: Net-(U9B--) -> Net-(U10B--)
- R53 pad 1: /HV_ON -> /+HV
- R53 pad 2: /20V_ON -> /+50V
- R54 pad 1: /+HV -> /HV_ON
- R54 pad 2: /+50V -> /50V_ON
- R56 pad 1: /HV_ON -> Net-(U16-RFB)
- R56 pad 2: /50V_ON -> Net-(U16-SW)
- R57 pad 1: /-HV -> /20V_FB
- R57 pad 2: /-20V -> /+20V
- R58 pad 1: Net-(U17-RFB) -> GND
- R58 pad 2: Net-(U17-SW) -> /50V_ON
- R59 pad 1: /20V_FB -> GND
- R59 pad 2: /+20V -> /20V_ON
- R60 pad 1: GND -> /-HV
- R60 pad 2: /50V_ON -> /-50V
- R61 pad 2: /20V_ON -> Net-(U16-RREF)
- R62 pad 1: /-HV -> GND
- R62 pad 2: /-50V -> /20V_FB
- R63 pad 1: GND -> Net-(U17-STAT)
- R63 pad 2: Net-(U17-RREF) -> Net-(D13-K)
- R64 pad 2: /20V_FB -> Net-(SW1-C)
- R65 pad 1: Net-(U18-STAT) -> GND
- R65 pad 2: Net-(D12-K) -> Net-(D14-K)
- R66 pad 1: GND -> Net-(U17-PROG)
- R66 pad 2: Net-(SW1-C) -> GND
- U10 pad 2: Net-(D4-K) -> /Z_ON
- U10 pad 3: /E1_Pre -> /Z_ON
- U10 pad 4: /-HV -> GND
- U10 pad 5: unconnected-(U10-Status-Pad5) -> Net-(U10B--)
- U10 pad 6: Net-(D4-K) -> /Z2
- U10 pad 7: /+HV -> +3.3V
- U10 pad 8: /Z_ON -> /Z1
- U10 pad 9: /-HV -> Net-(U10A--)
- U16 pad 1: Net-(U16-SW) -> /50V_ON
- U16 pad 2: GND -> Net-(U16-INTVCC)
- U16 pad 3: /20V_FB -> /V_ON
- U16 pad 4: /20V_ON -> GND
- U16 pad 5: /V_ON -> Net-(U16-SW)
- U17 pad 1: /50V_ON -> Net-(U17-STAT)
- U17 pad 2: Net-(U17-INTVCC) -> GND
- U17 pad 3: /V_ON -> /VBAT
- U17 pad 4: GND -> /V_USB
- U17 pad 5: Net-(U17-SW) -> Net-(U17-PROG)
- U9 pad 1: /Z1 -> GND
- U9 pad 2: Net-(U9A--) -> Net-(D4-K)
- U9 pad 3: GND -> /E1_Pre
- U9 pad 4: GND -> /-HV
- U9 pad 5: GND -> unconnected-(U9-Status-Pad5)
- U9 pad 6: Net-(U9B--) -> Net-(D4-K)
- U9 pad 7: /Z2 -> /+HV
- U9 pad 8: +3.3V -> /Z_ON
- U9 pad 9: (no net) -> /-HV
- Y1 pad 2: Net-(U5-XC1) -> GND
- Y1 pad 3: (no net) -> Net-(U5-XC1)
- Y1 pad 4: (no net) -> GND
Other:
- board outline added: 71.1 x 141 mm

Commit message: Updated 50V cap values and size
Parts:
- C38, C41: value C_Polarized_US -> 10uF, 100V electrolytic; footprint Capacitor_THT:CP_Radial_D12.5mm_P5.00mm -> Capacitor_THT:CP_Radial_D6.3mm_P2.50mm
- moved TP23 212.3 mm to (125.7, 249.9)
- moved TP24 212.3 mm to (125.7, 254.0)
- moved TP25 212.3 mm to (129.8, 225.7)
- moved TP27 212.3 mm to (129.8, 233.8)
- moved S1 202.4 mm to (142.3, 248.4)
- moved C27 192.0 mm to (131.6, 264.2)
- moved C28 192.0 mm to (156.4, 253.2)
- moved R43 192.0 mm to (143.1, 262.3)
- moved U13 176.1 mm to (154.1, 265.1)
- moved R56 156.6 mm to (-21.9, -41.9)
- moved R61 156.6 mm to (-21.9, -39.0)
- moved C47 146.9 mm to (0.78, -43.2)
- moved C46 146.9 mm to (0.78, -45.7)
- moved R58 146.9 mm to (-13.6, -36.0)
- moved R49 138.2 mm to (37.7, -54.6)
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
Commit message: Some lazy Saturday floorplanning on the layout
Parts:
- moved TP1 382.4 mm to (405.6, 82.9)
- moved TP2 382.4 mm to (405.6, 87.0)
- moved TP7 347.1 mm to (367.0, 124.2)
- moved TP8 347.1 mm to (367.0, 128.3)
- moved TP9 347.1 mm to (371.1, 99.9)
- moved TP10 327.8 mm to (358.1, 40.7)
- moved TP15 327.8 mm to (358.1, 61.0)
- moved TP16 326.7 mm to (356.9, 73.7)
- moved TP18 311.2 mm to (342.9, 78.5)
- moved TP19 311.2 mm to (342.9, 82.5)
- moved TP4 309.2 mm to (335.3, 55.9)
- moved TP32 308.0 mm to (307.3, 85.1)
- moved TP5 304.5 mm to (330.2, 68.6)
- moved TP3 300.8 mm to (326.4, 62.2)
- moved TP35 294.9 mm to (198.1, 124.5)
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Connections:
- U12 pad 3: /E1_Pre -> /E2_Pre
Other:
- copper layers 2 -> 4

Commit message: Started doing proper layout
Parts:
- removed TP40: TestPoint, TestPoint:TestPoint_Pad_D2.0mm
- added L4: 2.7nH, 5%, Inductor_SMD:L_0402_1005Metric, F.Cu at (261.6, 149.9)
- added L5: 1.8nH, 5%, Inductor_SMD:L_0402_1005Metric, F.Cu at (260.9, 148.3)
- moved TP1 201.8 mm to (205.7, 55.1)
- moved TP9 172.3 mm to (205.7, 51.6)
- moved TP2 156.7 mm to (248.9, 87.1)
- moved TP7 140.2 mm to (246.3, 52.8)
- moved TP8 140.2 mm to (246.3, 56.9)
- moved TP6 137.9 mm to (200.6, 69.3)
- moved TP4 131.9 mm to (205.7, 80.8)
- moved TP26 131.7 mm to (262.9, 134.6)
- moved TP21 129.9 mm to (245.1, 134.6)
- moved TP20 126.2 mm to (243.8, 124.5)
- moved TP25 125.4 mm to (219.7, 127.0)
- moved TP27 123.9 mm to (224.8, 138.4)
- moved TP16 121.7 mm to (237.5, 97.3)
- moved TP5 117.3 mm to (213.3, 59.2)
- moved TP3 116.1 mm to (214.6, 93.5)
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Connections:
- AT1 pad 1: /RF_ANT -> Net-(AT1-Pad1)
Routing:
- net GND: track 0.00 -> 35.1 mm, vias 0 -> 31
- net /V_ON: track 0.00 -> 32.5 mm, vias 0 -> 3
- net +3.3V: track 0.00 -> 27.5 mm, vias 0 -> 4
- net /V_USB: track 0.00 -> 23.2 mm
- net /HV_ON: track 0.00 -> 22.8 mm
- net /EmStop: track 0.00 -> 16.2 mm
- net /VBAT: track 0.00 -> 15.8 mm, vias 0 -> 3
- net /RF_ANT: track 0.00 -> 9.63 mm
- net Net-(U16-RREF): track 0.00 -> 8.22 mm
- net Net-(J3-CC2): track 0.00 -> 8.12 mm
- net Net-(U14-FB): track 0.00 -> 7.53 mm
- net Net-(J1-SWCLK/TCK): track 0.00 -> 6.82 mm
- net Net-(U5-XC1): track 0.00 -> 6.64 mm
- net /RF_MCU: track 0.00 -> 6.24 mm
- net Net-(U5-XC2): track 0.00 -> 6.02 mm
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- added copper zone on F.Cu, net +3.3V
- added copper zone on F.Cu, net /+20V
- added copper zone on F.Cu, net /+50V
- added copper zone on F.Cu, net /-20V
- added copper zone on F.Cu, net /-50V
- added copper zone on F.Cu, net /20V_FB
- added copper zone on F.Cu, net /VBAT
- added copper zone on F.Cu, net /V_ON
- added copper zone on F.Cu, net /V_USB
- added copper zone on F.Cu, net GND
- added copper zone on F.Cu, net Net-(U14-L)
- added copper zone on F.Cu, net Net-(U15-SW)
- added copper zone on F.Cu, net Net-(U16-SW)
Other:
- board size 71.1 x 141 mm -> 69.9 x 118.7 mm
- board text added: "Add Headers for Outputs Add hatches for hand soldered components After deciding stackup, need to go through and calculate all 50 Ohm lines (USB data and RF antenna)"

Commit message: First draft of layout, still has work to be done
Parts:
- added J5: Conn_01x03_Pin, Connector_PinHeader_2.54mm:PinHeader_1x03_P2.54mm_Vertical, F.Cu at (219.7, 36.8)
- added R67: 100k, Resistor_SMD:R_0402_1005Metric, F.Cu at (206.9, 154.1)
- added R68: 100k, Resistor_SMD:R_0402_1005Metric, F.Cu at (206.9, 156.0)
- moved TP8 75.0 mm to (219.7, 127.0)
- moved U12 20.9 mm to (257.2, 92.0)
- moved U9 20.9 mm to (249.6, 92.0)
- moved TP15 20.6 mm to (252.7, 81.3)
- moved C23 20.4 mm to (217.1, 68.1), turned to 90 degrees
- moved TP5 20.2 mm to (218.4, 78.7)
- moved TP25 19.4 mm to (238.8, 123.2)
- moved J2 19.2 mm to (226.1, 69.2)
- moved TP2 19.1 mm to (229.9, 85.1)
- moved TP17 18.9 mm to (259.1, 81.3)
- moved TP23 18.3 mm to (238.8, 138.7)
- moved TP19 18.1 mm to (240.2, 78.2)
- moved C16 17.4 mm to (225.8, 84.0)
- moved C15 17.4 mm to (225.8, 80.8)
- moved R21 16.8 mm to (219.2, 66.7), turned to -90 degrees
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Connections:
- U5 pad H2: unconnected-(U5-P0.27-PadH2) -> /Batt_Measure
Routing:
- net GND: track 35.1 -> 159.5 mm, vias 31 -> 75
- net /I2C_SCL: track 0.00 -> 94.3 mm, vias 0 -> 5
- net /I2C_SDA: track 2.07 -> 94.4 mm, vias 0 -> 4
- net /C2A_ON: track 0.00 -> 78.8 mm, vias 0 -> 3
- net /C1A_ON: track 0.00 -> 70.6 mm, vias 0 -> 2
- net /C2C_ON: track 0.00 -> 68.3 mm, vias 0 -> 2
- net /Z_ON: track 0.00 -> 65.4 mm, vias 0 -> 4
- net /C1C_ON: track 0.00 -> 63.9 mm, vias 0 -> 2
- net /V_ON: track 32.5 -> 95.9 mm, vias 3 -> 11
- net +3.3V: track 27.5 -> 77.3 mm, vias 4 -> 20
- net Net-(D4-K): track 0.00 -> 47.3 mm
- net Net-(D6-K): track 0.00 -> 42.4 mm
- net /E1_Pre: track 0.00 -> 41.5 mm, vias 0 -> 2
- net /VBAT: track 15.8 -> 53.2 mm, vias 3 -> 5
- net /EmStop: track 16.2 -> 52.4 mm, vias 0 -> 2
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- added copper zone on In2.Cu, net +3.3V
- added copper zone on In1.Cu, net /+HV
- added copper zone on In2.Cu, net /-HV
- added copper zone on F.Cu, net /E1
- added copper zone on F.Cu, net /E1_Pre
- added copper zone on F.Cu, net /E2_Pre
- added copper zone on B.Cu, net GND
- added copper zone on In1.Cu, net GND
Other:
- board size 69.9 x 118.7 mm -> 69.9 x 100.9 mm

Commit message: Added 3D model for transformer
Parts:
- moved J5 36.3 mm to (198.1, 66.0)
Changed lines of the file:
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@@
 		)
 		(embedded_fonts no)
+		(model "/Users/alexbaldwin/Desktop/Unnamed-Cube.step"
+			(offset
+				(xyz -6.5 -6.5 0)
+			)
+			(scale
+				(xyz 1 1 1)
+			)
+			(rotate
+				(xyz -0 -0 -0)
+			)
+		)
 	)
 	(footprint "TestPoint:TestPoint_Pad_D2.0mm"
@@
 	(footprint "Connector_PinHeader_2.54mm:PinHeader_1x03_P2.54mm_Vertical"
 		(layer "F.Cu")
-		(at 219.71 36.83 90)
+		(at 198.12 66.04 90)
 		(descr "Through hole straight pin header, 1x03, 2.54mm pitch, single row")
 		(tags "Through hole pin header THT 1x03 2.54mm single row")
