File: hardware/OpenAVNS KiCad Project.kicad_sch (KiCad schematic)
At the start: 211 parts, among them J1 Conn_ARM_JTAG_SWD_10, J2 AudioPlug3, J3 Conn_02x02_Top_Bottom, J4 Conn_01x02_Pin, J5 Conn_01x03_Pin, J6 Conn_01x01_Pin, J7 2171790001, J8 Conn_02x02_Top_Bottom, J9 Conn_02x02_Top_Bottom, Q1 BCV62, Q2 BC847, Q3 BC857, Q4 BCV61, Q5 BCV62, Q6 BC847, Q7 BC857, Q8 BCV61, SW1 SW_SPDT, T1 Wurth 750315839 - 1:10, 40uH, U10 TLV9062, U11 LIS2DH12, U12 OPA455, U13 74AUC1G74, U14 TPS61200DRC, U15 LT1615ES5_TRPBF, U16 LT8304IS8E_PBF, U17 MCP73831-2-OT, U18 TS5A3159DCKR, U19 TS5A3159DCKR, U2 TLV9004xRUCR, U20 TS5A3159DCKR, U21 TS5A3159DCKR, U3 MCP4725xxx-xCH, U5 nRF52840, U7 MCP4725xxx-xCH, U9 OPA455, Y1 32MHz - X322532MOB4SI

Commit message: Updated PCBA design based on debugging results - untested, still needs more work and simulation
Parts:
- removed C27: 100nF, Capacitor_SMD:C_0402_1005Metric, symbol Device:C
- removed C28: 10uF, Capacitor_SMD:C_0603_1608Metric, symbol Device:C
- removed D4, D6: SS3200, Diode_SMD:D_SMA, symbol Diode:SS3200
- removed R41, R45: 100k, Resistor_SMD:R_0402_1005Metric, symbol Device:R_US
- removed R46: 619 Ohm, Resistor_SMD:R_1206_3216Metric, symbol Device:R_US
- removed TP22, TP23, TP27: TestPoint, TestPoint:TestPoint_Pad_D2.0mm, symbol Connector:TestPoint
- removed U12: OPA455, Package_SO:TI_SO-PowerPAD-8_ThermalVias, symbol Amplifier_Operational:OPA455
- removed U13: 74AUC1G74, Package_DFN_QFN:Texas_UQFN-8_1.5x1.5mm_P0.5mm, symbol 74xGxx:74AUC1G74
- added C50, C51, C52, C53, C54, C55, C56, C57: 100nF, Capacitor_SMD:C_0402_1005Metric, symbol Device:C
- added R49, R52, R53, R54: 100k, Capacitor_SMD:C_0402_1005Metric, symbol Device:R_US
- added R55, R60, R73, R74: 500 Ohm, Capacitor_SMD:C_0402_1005Metric, symbol Device:R_US
- added R69, R70, R71, R72: 100k, Resistor_SMD:R_0805_2012Metric_Pad1.20x1.40mm_HandSolder, symbol Device:R_US
- added U22, U23, U24, U25, U26, U27, U28: TS5A3159DCKR, Footprints:SOT65P210X110-6N, symbol TS5A3159DCKR:TS5A3159DCKR
- R11, R14: value 0 Ohm -> 1M; footprint Resistor_SMD:R_0603_1608Metric_Pad0.98x0.95mm_HandSolder -> Capacitor_SMD:C_0402_1005Metric
- R17, R18: value 0 Ohm -> 100k; footprint Resistor_SMD:R_0603_1608Metric_Pad0.98x0.95mm_HandSolder -> Capacitor_SMD:C_0402_1005Metric
- R25, R26: value 22 Ohm -> 33 Ohm
- R35: value 100k -> 1M
- R40: value 619 Ohm -> 811 Ohm
- R44: value 10k -> 100k; footprint Resistor_SMD:R_1206_3216Metric -> Resistor_SMD:R_0402_1005Metric
- R56: value 100k -> 200k
Connections:
- net HV_EN is gone; now on net HV_ON: U5.AC19 (P0.23)
- net +20V: now also R69.2
- net +3.3V: now also C50.1, C51.1, C52.1, C53.1, C54.1, C55.1, C57.1, U22.5, U23.5, U24.5, U25.5, U26.5, U27.5, U28.5; no longer R35.2
- net +50V: now also R71.2
- net -20V: now also R70.1
- net -50V: now also R72.1
- net C1A_ON: now also R11.2
- net C1C_ON: now also R14.2
- net C1_Anodic: now also U25.4; no longer R11.2
- net C1_Cathodic: now also U24.4; no longer R14.2
- net C2A_ON: now also R17.2
- net C2C_ON: now also R18.2
- net C2_Anodic: now also U23.4; no longer R17.2
- net C2_Cathodic: now also U22.4; no longer R18.2
- net E1_Pre: now also U26.4, U28.3; no longer R11.1, R14.1, U9.3 (+)
- net E2_Pre: now also U27.4, U28.1; no longer R17.1, R18.1
- net GND: now also R11.1, R14.1, R17.1, R18.1, R44.1, C50.2, C51.2, C52.2, C53.2, C54.2, C55.2, C57.2, R49.1, R52.1, R53.1, R54.1, R55.1, R60.1, R69.1, R70.2, R71.1, R72.2, R73.1, R74.1, U22.2, U23.2, U24.2, U25.2, U26.1, U26.2, U27.1, U27.2, U28.2; no longer U10.10 (+), U10.4 (+)
- net at R38.1, TP20.1: now also U9.2 (-), U9.6 (OUT)
- net at R38.2, R40.1: now also R35.2; no longer R39.2
- net at R34.2, R39.1, U10.9 (-): now also C56.1; no longer R35.1
- net at R30.1, U2.11 (+): now also U21.1; no longer U21.3
- net at R42.1: now also R44.2, U10.4 (+); no longer U10.5 (-)
- net at R23.2, U2.9 (+): now also U20.1; no longer U20.3
- net E2_GND_SW: now reaches U5.R24 (P1.06)
- net E2_GND_SW: now also U27.6
- net E1_GND_SW: now reaches U5.T23 (P1.05)
- net E1_GND_SW: now also U26.6
- net C2C_Out_Sw: now reaches U5.U24 (P1.04)
- net C2C_Out_Sw: now also R54.2, U22.6
- net C2A_Out_Sw: now reaches U5.V23 (P1.03)
- net C2A_Out_Sw: now also R53.2, U23.6
- net C1C_Out_Sw: now reaches U5.W24 (P1.02)
- net C1C_Out_Sw: now also R52.2, U24.6
- net C1A_Out_Sw: now reaches U5.Y23 (P1.01)
- net C1A_Out_Sw: now also R49.2, U25.6
- net at R9.1, U2.4 (+): now also U19.1; no longer U19.3
- net at R4.2, U2.2 (+): now also U18.1; no longer U18.3
- net Z1 renamed Z_OUT
- net Z_OUT: no longer U5.A12 (AIN0/P0.02)
- net Z2 renamed Z_1V65
- net Z_1V65: now also R39.2, U10.10 (+), U10.5 (-); no longer U5.B13 (AIN1/P0.03)
- new net: R74.2, U25.3
- new net: R60.2, U23.3
- new net: C56.2, R35.1
- new net: U28.4, U9.3 (+)
- new net: R73.2, U24.3
- new net: R55.2, U22.3
- new net C1_Out: U24.1, U25.1, U26.3
- new net C2_Out: U22.1, U23.1, U27.3
- new net Z_Out: U5.A12 (AIN0/P0.02)
- new net Z_SW: U28.6, U5.B13 (AIN1/P0.03)
Other:
- note added: "Empirically, 100k for Rfb led to +/-25V. Increasing to 200k to get +/-50V (untested)"
- note added: "HV Selection"
- note removed: "For -50V scaling, ratio should be 6.19k to 100k For -20V scaling, ratio should be 14.16k to 100k"
- note removed: "HV Selection Resistors"
- note removed: "HV Shutdown on Button"
- moved on the sheet: C29, C30, H1, H2, H3, H4, R34, R43, S1, TP21, TP25, TP34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

Commit message: Routed schematic with new output switches, new impedance circuit
Connections:
- net Z_Out is gone; now on net Z_OUT: U5.A12 (AIN0/P0.02)
Changed lines of the file:
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@@
 		)
 	)
-	(label "Z_Out"
+	(label "Z_OUT"
 		(at 180.34 105.41 0)
 		(effects
